File: Hardware/tkl_keyboard/tkl_keyboard_placement.kicad_pcb (KiCad board)
At the start: 2 copper layers, 3.4 x 3 mm, 468 parts, among them J1 USB_C_Receptacle_USB2.0, J2 USB_C_Receptacle_USB2.0, J3 USB_C_Receptacle_USB2.0, J4 USB_C_Receptacle_USB2.0, J5 Conn_02x03_Odd_Even, J6 Conn_01x04_Female, SW1 SW_Push, SW10 K33, SW11 K49, SW12 K64, SW13 K2, SW14 K18, SW15 K34, SW16 K50, SW17 K65, SW18 K78, SW19 K3, SW2 K0, SW20 K19, SW21 K35, SW22 K51, SW23 K66, SW24 K4, SW25 K20, SW26 K36, SW27 K52, SW28 K67, SW29 K79, SW3 K16, SW30 K5, SW31 K21, SW32 K37, SW33 K53, SW34 K68, SW35 K6, SW36 K22, SW37 K38, SW38 K54, SW39 K69, SW4 K32, SW40 K80, SW41 K7, SW42 K23, SW43 K39, SW44 K55, SW45 K70, SW46 K8, SW47 K24, SW48 K40, SW49 K56, SW5 K48, SW50 K71, SW51 K81, SW52 K9, SW53 K25, SW54 K41, SW55 K57, SW56 K72, SW57 K82, SW58 K10, SW59 K26, SW6 K63, SW60 K42, SW61 K58, SW62 K73, SW63 K83, SW64 K11, SW65 K27, SW66 K43, SW67 K59, SW68 K74, SW69 K84, SW7 K77, SW70 K12, SW71 K28, SW72 K44, SW73 K60, SW74 K75, SW75 K85, SW76 K13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

Commit message: LEDs and diodes routed
Parts:
- added U7: CD74HC238, Package_SO:SOIC-16_3.9x9.9mm_P1.27mm, B.Cu at (110.8, 76.0)
- added U8: CD74HC238, Package_SO:SOIC-16_3.9x9.9mm_P1.27mm, B.Cu at (300.8, 71.4)
- C1, C10, C100, C102, C103, C104, C105, C106, C107, C108, C109, C11, C110, C111, C112, C113, C115, C12, C13, C14, C15, C16, C17, C18, C19, C2, C20, C21, C22, C24, C26, C27, C28, C29, C30, C33, C34, C35, C36, C37, C38, C40, C41, C43, C47, C48, C49, C50, C51, C52, C53, C54, C55, C56, C57, C58, C60, C61, C62, C63, C64, C65, C66, C67, C68, C69, C70, C71, C73, C76, C77, C78, C79, C80, C81, C82, C83, C84, C85, C86, C89, C9, C90, C91, C92, C93, C94, C95, C96, C97, C98, C99, R20, R21, R23, R38, R39, U6, X1, X2: moved to B.Cu
- D14: value UG_LED_2 -> UG_0
- D15: value UG_LED_8 -> UG_6
- D160: value UG_LED_12 -> UG_10
- D167: value UG_LED_13 -> UG_11
- D174: value UG_LED_14 -> UG_12
- D180: value UG_LED_15 -> UG_13
- D2: value UG_LED_6 -> UG_4
- D21: value UG_LED_3 -> UG_1
- D22: value UG_LED_9 -> UG_7
- D28: value UG_LED_4 -> UG_2
- D29: value UG_LED_10 -> UG_8
- D30: value UG_LED_5 -> UG_3
- D31: value UG_LED_11 -> UG_9
- D8: value UG_LED_7 -> UG_5
- moved SW92 383.4 mm to (368.3, 81.8), turned to 270 degrees
- moved R37 379.4 mm to (366.3, 73.5), turned to 270 degrees
- moved SW91 372.9 mm to (349.2, 81.8), turned to 270 degrees
- moved R34 368.2 mm to (364.7, 73.5), turned to 270 degrees
- moved H2 357.8 mm to (374.6, 79.4)
- moved R36 343.0 mm to (346.9, 73.3), turned to 270 degrees
- moved R32 337.3 mm to (324.8, 73.8), turned to 270 degrees
- moved R35 336.5 mm to (322.3, 73.8), turned to 270 degrees
- moved SW90 332.5 mm to (330.2, 81.8), turned to 270 degrees
- moved R33 329.1 mm to (345.5, 73.4), turned to 270 degrees
- moved H3 320.1 mm to (374.6, 199.2)
- moved FB3 306.8 mm to (246.5, 69.6), turned to 90 degrees
- moved C4 305.8 mm to (253.0, 66.0), turned to 180 degrees
- moved C2 304.6 mm to (241.4, 62.9), turned to 90 degrees
- moved J1 301.2 mm to (242.8, 67.2), turned to 180 degrees
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Connections:
- D106 pad 2: Net-(D106-Pad2) -> ENC_ROW[0]
- D111 pad 2: Net-(D111-Pad2) -> ENC_ROW[1]
- D116 pad 2: Net-(D116-Pad2) -> ENC_ROW[2]
- D183 pad 2: Net-(D178-Pad4) -> Net-(D12-Pad4)
- D186 pad 4: Net-(D182-Pad2) -> Net-(D186-Pad4)
- D19 pad 2: Net-(D12-Pad4) -> Net-(D183-Pad4)
- D190 pad 2: Net-(D190-Pad2) -> Net-(D178-Pad4)
- D193 pad 2: Net-(D183-Pad4) -> Net-(D186-Pad4)
- D193 pad 4: Net-(D190-Pad2) -> Net-(D182-Pad2)
- J2 pad A6: /USB Downstrem 0/USBD+ -> /USB Downstream 0/USBD+
- J2 pad A7: /USB Downstrem 0/USBD- -> /USB Downstream 0/USBD-
- J2 pad B6: /USB Downstrem 0/USBD+ -> /USB Downstream 0/USBD+
- J2 pad B7: /USB Downstrem 0/USBD- -> /USB Downstream 0/USBD-
- R12 pad 1: /USB Downstrem 0/USBD+ -> /USB Downstream 0/USBD+
- R13 pad 1: /USB Downstrem 0/USBD- -> /USB Downstream 0/USBD-
- SW76 pad 1: Net-(D106-Pad2) -> ENC_ROW[0]
- SW76 pad 2: /Column Decoder/COL[13] -> ENC_COL[0]
- SW77 pad 2: /Column Decoder/COL[13] -> ENC_COL[0]
- SW78 pad 2: /Column Decoder/COL[13] -> ENC_COL[0]
- SW79 pad 2: /Column Decoder/COL[13] -> ENC_COL[0]
- SW80 pad 2: /Column Decoder/COL[13] -> ENC_COL[0]
- SW81 pad 1: Net-(D111-Pad2) -> ENC_ROW[1]
- SW81 pad 2: /Column Decoder/COL[14] -> ENC_COL[1]
- SW82 pad 2: /Column Decoder/COL[14] -> ENC_COL[1]
- SW83 pad 2: /Column Decoder/COL[14] -> ENC_COL[1]
- SW84 pad 2: /Column Decoder/COL[14] -> ENC_COL[1]
- SW85 pad 2: /Column Decoder/COL[14] -> ENC_COL[1]
- SW86 pad 1: Net-(D116-Pad2) -> ENC_ROW[2]
- SW86 pad 2: /Column Decoder/COL[15] -> ENC_COL[2]
- SW87 pad 2: /Column Decoder/COL[15] -> ENC_COL[2]
- SW88 pad 2: /Column Decoder/COL[15] -> ENC_COL[2]
- SW89 pad 2: /Column Decoder/COL[15] -> ENC_COL[2]
- SW93 pad 2: /Column Decoder/COL[14] -> ENC_COL[1]
- U3 pad 1: USB_D1- -> /USB Downstream 0/USBD-
- U3 pad 3: USB_D2+ -> /USB Downstream 1/USBD+
- U3 pad 4: USB_D2- -> /USB Downstream 1/USBD-
- U3 pad 6: USB_D1+ -> /USB Downstream 0/USBD+
- U5 pad 3: USB_D3+ -> /USB Downstream 2/USBD-
- U5 pad 4: USB_D3- -> /USB Downstream 2/USBD+
Routing:
- net ENC_ROW[2]: track 0.00 -> 5.66 mm
- net ENC_ROW[0]: track 0.00 -> 5.42 mm
- net ENC_ROW[1]: track 0.00 -> 5.40 mm
- net Net-(D97-Pad2): track 0.00 -> 3.55 mm
- net Net-(D94-Pad2): track 0.00 -> 3.55 mm
- net Net-(D119-Pad2): track 0.00 -> 3.55 mm
- net Net-(D115-Pad2): track 0.00 -> 3.55 mm
- net Net-(D100-Pad2): track 0.00 -> 3.55 mm
- net Net-(D117-Pad2): track 0.00 -> 3.55 mm
- net Net-(D112-Pad2): track 0.00 -> 3.55 mm
- net Net-(D91-Pad2): track 0.00 -> 3.55 mm
- net Net-(D87-Pad2): track 0.00 -> 3.55 mm
- net Net-(D81-Pad2): track 0.00 -> 3.55 mm
- net Net-(D79-Pad2): track 0.00 -> 3.55 mm
- net Net-(D76-Pad2): track 0.00 -> 3.55 mm
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- added copper zone on F.Cu, net +5V
- added copper zone on B.Cu, net GND
Other:
- board size 3.4 x 3 mm -> 358.8 x 141.1 mm
