File: Hardware/tkl_keyboard/tkl_keyboard.kicad_pcb (KiCad board)
At the start: 2 copper layers, 3.4 x 3 mm, 468 parts, among them J1 USB_C_Receptacle_USB2.0, J2 USB_C_Receptacle_USB2.0, J3 USB_C_Receptacle_USB2.0, J4 USB_C_Receptacle_USB2.0, J5 Conn_02x03_Odd_Even, J6 Conn_01x04_Female, SW1 SW_Push, SW10 K33, SW11 K49, SW12 K64, SW13 K2, SW14 K18, SW15 K34, SW16 K50, SW17 K65, SW18 K78, SW19 K3, SW2 K0, SW20 K19, SW21 K35, SW22 K51, SW23 K66, SW24 K4, SW25 K20, SW26 K36, SW27 K52, SW28 K67, SW29 K79, SW3 K16, SW30 K5, SW31 K21, SW32 K37, SW33 K53, SW34 K68, SW35 K6, SW36 K22, SW37 K38, SW38 K54, SW39 K69, SW4 K32, SW40 K80, SW41 K7, SW42 K23, SW43 K39, SW44 K55, SW45 K70, SW46 K8, SW47 K24, SW48 K40, SW49 K56, SW5 K48, SW50 K71, SW51 K81, SW52 K9, SW53 K25, SW54 K41, SW55 K57, SW56 K72, SW57 K82, SW58 K10, SW59 K26, SW6 K63, SW60 K42, SW61 K58, SW62 K73, SW63 K83, SW64 K11, SW65 K27, SW66 K43, SW67 K59, SW68 K74, SW69 K84, SW7 K77, SW70 K12, SW71 K28, SW72 K44, SW73 K60, SW74 K75, SW75 K85, SW76 K13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

Commit message: LEDs and diodes routed
Parts:
- added U7: CD74HC238, Package_SO:SOIC-16_3.9x9.9mm_P1.27mm, B.Cu at (110.8, 76.0)
- added U8: CD74HC238, Package_SO:SOIC-16_3.9x9.9mm_P1.27mm, B.Cu at (300.8, 71.4)
- C1, C10, C100, C102, C103, C104, C105, C106, C107, C108, C109, C11, C110, C111, C112, C113, C115, C12, C13, C14, C15, C16, C17, C18, C19, C2, C20, C21, C22, C24, C26, C27, C28, C29, C30, C33, C34, C35, C36, C37, C38, C40, C41, C43, C47, C48, C49, C50, C51, C52, C53, C54, C55, C56, C57, C58, C60, C61, C62, C63, C64, C65, C66, C67, C68, C69, C70, C71, C73, C76, C77, C78, C79, C80, C81, C82, C83, C84, C85, C86, C89, C9, C90, C91, C92, C93, C94, C95, C96, C97, C98, C99, R21, R23, R38, R39, U6, X1, X2: moved to B.Cu
- D14: value UG_LED_2 -> UG_0
- D15: value UG_LED_8 -> UG_6
- D160: value UG_LED_12 -> UG_10
- D167: value UG_LED_13 -> UG_11
- D174: value UG_LED_14 -> UG_12
- D180: value UG_LED_15 -> UG_13
- D2: value UG_LED_6 -> UG_4
- D21: value UG_LED_3 -> UG_1
- D22: value UG_LED_9 -> UG_7
- D28: value UG_LED_4 -> UG_2
- D29: value UG_LED_10 -> UG_8
- D30: value UG_LED_5 -> UG_3
- D31: value UG_LED_11 -> UG_9
- D8: value UG_LED_7 -> UG_5
- moved SW92 383.4 mm to (368.3, 81.8), turned to 270 degrees
- moved R37 379.4 mm to (366.3, 73.5), turned to 270 degrees
- moved SW91 372.9 mm to (349.2, 81.8), turned to 270 degrees
- moved R34 368.2 mm to (364.7, 73.5), turned to 270 degrees
- moved H2 364.9 mm to (374.6, 64.3)
- moved R36 343.0 mm to (346.9, 73.3), turned to 270 degrees
- moved R32 337.3 mm to (324.8, 73.8), turned to 270 degrees
- moved R35 336.5 mm to (322.3, 73.8), turned to 270 degrees
- moved SW90 332.5 mm to (330.2, 81.8), turned to 270 degrees
- moved R33 329.1 mm to (345.5, 73.4), turned to 270 degrees
- moved H3 320.1 mm to (374.6, 199.2)
- moved FB3 306.8 mm to (246.5, 69.6), turned to 90 degrees
- moved C4 305.8 mm to (253.0, 66.0), turned to 180 degrees
- moved C2 304.6 mm to (241.4, 62.9), turned to 90 degrees
- moved J1 301.2 mm to (242.8, 67.2), turned to 180 degrees
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Connections:
- D106 pad 2: Net-(D106-Pad2) -> ENC_ROW[0]
- D111 pad 2: Net-(D111-Pad2) -> ENC_ROW[1]
- D116 pad 2: Net-(D116-Pad2) -> ENC_ROW[2]
- D121 pad 2: Net-(D11-Pad4) -> Net-(D121-Pad2)
- D17 pad 2: Net-(D17-Pad2) -> Net-(D11-Pad4)
- D17 pad 4: Net-(D17-Pad4) -> Net-(D121-Pad2)
- D183 pad 2: Net-(D178-Pad4) -> Net-(D12-Pad4)
- D186 pad 4: Net-(D182-Pad2) -> Net-(D186-Pad4)
- D19 pad 2: Net-(D12-Pad4) -> Net-(D183-Pad4)
- D190 pad 2: Net-(D190-Pad2) -> Net-(D178-Pad4)
- D193 pad 2: Net-(D183-Pad4) -> Net-(D186-Pad4)
- D193 pad 4: Net-(D190-Pad2) -> Net-(D182-Pad2)
- D25 pad 4: Net-(D17-Pad2) -> Net-(D25-Pad4)
- D5 pad 2: Net-(D17-Pad4) -> Net-(D25-Pad4)
- J2 pad A6: /USB Downstrem 0/USBD+ -> /USB Downstream 0/USBD+
- J2 pad A7: /USB Downstrem 0/USBD- -> /USB Downstream 0/USBD-
- J2 pad B6: /USB Downstrem 0/USBD+ -> /USB Downstream 0/USBD+
- J2 pad B7: /USB Downstrem 0/USBD- -> /USB Downstream 0/USBD-
- R12 pad 1: /USB Downstrem 0/USBD+ -> /USB Downstream 0/USBD+
- R13 pad 1: /USB Downstrem 0/USBD- -> /USB Downstream 0/USBD-
- SW76 pad 1: Net-(D106-Pad2) -> ENC_ROW[0]
- SW76 pad 2: /Column Decoder/COL[13] -> ENC_COL[0]
- SW77 pad 2: /Column Decoder/COL[13] -> ENC_COL[0]
- SW78 pad 2: /Column Decoder/COL[13] -> ENC_COL[0]
- SW79 pad 2: /Column Decoder/COL[13] -> ENC_COL[0]
- SW80 pad 2: /Column Decoder/COL[13] -> ENC_COL[0]
- SW81 pad 1: Net-(D111-Pad2) -> ENC_ROW[1]
- SW81 pad 2: /Column Decoder/COL[14] -> ENC_COL[1]
- SW82 pad 2: /Column Decoder/COL[14] -> ENC_COL[1]
- SW83 pad 2: /Column Decoder/COL[14] -> ENC_COL[1]
- SW84 pad 2: /Column Decoder/COL[14] -> ENC_COL[1]
- SW85 pad 2: /Column Decoder/COL[14] -> ENC_COL[1]
- SW86 pad 1: Net-(D116-Pad2) -> ENC_ROW[2]
- SW86 pad 2: /Column Decoder/COL[15] -> ENC_COL[2]
- SW87 pad 2: /Column Decoder/COL[15] -> ENC_COL[2]
- SW88 pad 2: /Column Decoder/COL[15] -> ENC_COL[2]
- SW89 pad 2: /Column Decoder/COL[15] -> ENC_COL[2]
- SW93 pad 2: /Column Decoder/COL[14] -> ENC_COL[1]
- U3 pad 1: USB_D1- -> /USB Downstream 0/USBD-
- U3 pad 3: USB_D2+ -> /USB Downstream 1/USBD+
- U3 pad 4: USB_D2- -> /USB Downstream 1/USBD-
- U3 pad 6: USB_D1+ -> /USB Downstream 0/USBD+
- U5 pad 3: USB_D3+ -> /USB Downstream 2/USBD-
- U5 pad 4: USB_D3- -> /USB Downstream 2/USBD+
Routing:
- net +5V: track 0.00 -> 364.5 mm, vias 0 -> 132
- net Net-(D178-Pad4): track 0.00 -> 102.7 mm, vias 0 -> 2
- net Net-(D29-Pad2): track 0.00 -> 86.0 mm, vias 0 -> 2
- net Net-(D160-Pad2): track 0.00 -> 83.7 mm, vias 0 -> 2
- net Net-(D22-Pad2): track 0.00 -> 78.2 mm, vias 0 -> 2
- net Net-(D160-Pad4): track 0.00 -> 68.6 mm, vias 0 -> 2
- net Net-(D177-Pad2): track 0.00 -> 56.6 mm, vias 0 -> 2
- net Net-(D15-Pad2): track 0.00 -> 52.2 mm, vias 0 -> 2
- net GND: track 0.00 -> 41.4 mm, vias 0 -> 27
- net Net-(D167-Pad2): track 0.00 -> 35.3 mm, vias 0 -> 2
- net Net-(D2-Pad2): track 0.00 -> 34.5 mm, vias 0 -> 2
- net Net-(D174-Pad2): track 0.00 -> 34.5 mm, vias 0 -> 2
- net Net-(D15-Pad4): track 0.00 -> 34.1 mm, vias 0 -> 2
- net Net-(D142-Pad4): track 0.00 -> 33.5 mm
- net Net-(D131-Pad4): track 0.00 -> 33.5 mm
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- added copper zone on F.Cu, net +5V
- added copper zone on B.Cu, net GND
Other:
- board size 3.4 x 3 mm -> 358.8 x 141.1 mm

Commit message: Switch matrix routed
Parts:
- FB1, R32, R33, R34, R35, R36, R37: moved to B.Cu
- X2: moved to F.Cu
- moved R16 89.1 mm to (113.3, 70.5), turned to 270 degrees
- moved R17 87.5 mm to (114.8, 70.5), turned to 270 degrees
- moved X2 75.5 mm to (205.6, 66.6), turned to 270 degrees
- moved C44 75.2 mm to (203.4, 79.1)
- moved C45 75.2 mm to (214.3, 66.8)
- moved C42 75.2 mm to (212.0, 79.2)
- moved C43 75.2 mm to (197.7, 71.5)
- moved R23 75.2 mm to (215.0, 76.1)
- moved U6 75.2 mm to (206.3, 71.5)
- moved C46 70.5 mm to (203.1, 73.7)
- moved R14 70.0 mm to (137.0, 70.4)
- moved R15 70.0 mm to (138.6, 70.4)
- moved J5 58.3 mm to (206.0, 48.9)
- moved R22 58.3 mm to (209.2, 56.1)
- moved SW1 58.3 mm to (212.3, 48.9)
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Connections:
- D42 pad 1: /Switches/ROW[4] -> /Switches/ROW[5]
- U7 pad 10: /Column Decoder/COL[2] -> /Column Decoder/COL[5]
- U7 pad 11: /Column Decoder/COL[3] -> /Column Decoder/COL[4]
- U7 pad 12: /Column Decoder/COL[4] -> /Column Decoder/COL[3]
- U7 pad 13: /Column Decoder/COL[5] -> /Column Decoder/COL[2]
- U7 pad 14: /Column Decoder/COL[6] -> /Column Decoder/COL[1]
- U7 pad 15: /Column Decoder/COL[7] -> /Column Decoder/COL[0]
- U7 pad 7: /Column Decoder/COL[0] -> /Column Decoder/COL[7]
- U7 pad 9: /Column Decoder/COL[1] -> /Column Decoder/COL[6]
- U8 pad 10: /Column Decoder/COL[10] -> ENC_COL[0]
- U8 pad 11: /Column Decoder/COL[11] -> /Column Decoder/COL[12]
- U8 pad 12: /Column Decoder/COL[12] -> /Column Decoder/COL[11]
- U8 pad 13: ENC_COL[0] -> /Column Decoder/COL[10]
- U8 pad 14: ENC_COL[1] -> /Column Decoder/COL[9]
- U8 pad 15: ENC_COL[2] -> /Column Decoder/COL[8]
- U8 pad 7: /Column Decoder/COL[8] -> ENC_COL[2]
- U8 pad 9: /Column Decoder/COL[9] -> ENC_COL[1]
Routing:
- net /Switches/ROW[1]: track 0.00 -> 341.6 mm, vias 0 -> 30
- net /Switches/ROW[0]: track 0.00 -> 334.2 mm
- net /Switches/ROW[5]: track 0.00 -> 331.9 mm, vias 0 -> 24
- net /Switches/ROW[3]: track 0.00 -> 327.5 mm, vias 0 -> 27
- net /Switches/ROW[2]: track 0.00 -> 326.4 mm
- net /Switches/ROW[4]: track 0.00 -> 299.6 mm
- net ENC_COL[0]: track 0.00 -> 167.8 mm, vias 0 -> 5
- net /Column Decoder/COL[11]: track 0.00 -> 151.3 mm, vias 0 -> 6
- net /Column Decoder/COL[10]: track 0.00 -> 145.3 mm, vias 0 -> 6
- net /Column Decoder/COL[12]: track 0.00 -> 143.8 mm, vias 0 -> 6
- net /Column Decoder/COL[9]: track 0.00 -> 141.7 mm, vias 0 -> 6
- net ENC_COL[1]: track 0.00 -> 132.1 mm, vias 0 -> 5
- net /Column Decoder/COL[8]: track 0.00 -> 121.7 mm, vias 0 -> 6
- net /Column Decoder/COL[6]: track 0.00 -> 121.6 mm, vias 0 -> 6
- net /Column Decoder/COL[2]: track 0.00 -> 114.9 mm, vias 0 -> 6
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
Commit message: Rows and columns routed to controller. Extended top board edge to fit OLED. Removed optional resistors around CMC.
Parts:
- removed R3, R4: OPT, resistor_smd:R_0603_1608Metric
- C45, FB2: moved to B.Cu
- J5: footprint Connector_PinHeader_2.54mm:PinHeader_2x03_P2.54mm_Vertical_SMD -> custom_footprint_library:ISP_POGO
- J6: footprint Connector_PinSocket_2.54mm:PinSocket_1x04_P2.54mm_Vertical -> custom_footprint_library:OLED_128_64
- moved C6 56.7 mm to (239.7, 46.7), turned to 270 degrees
- moved R10 54.5 mm to (238.1, 46.7), turned to 90 degrees
- moved R23 34.0 mm to (182.6, 66.0), turned to 180 degrees
- moved R26 32.1 mm to (107.1, 77.2)
- moved R38 31.9 mm to (213.2, 70.8)
- moved R39 31.9 mm to (213.2, 69.2)
- moved U4 31.9 mm to (213.2, 70.6)
- moved X1 31.9 mm to (216.8, 71.3)
- moved U7 31.6 mm to (105.3, 76.0)
- moved R25 31.2 mm to (105.4, 74.5)
- moved D14 31.1 mm to (71.4, 54.8)
- moved R5 31.1 mm to (220.2, 72.3)
- moved R6 31.1 mm to (220.2, 73.9)
- moved R24 31.1 mm to (103.7, 74.3)
- moved C42 31.1 mm to (185.6, 62.9), turned to 180 degrees
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Connections:
- net Net-(J1-PadA6) renamed /USB Upstream/CD+
- net Net-(J1-PadA7) renamed /USB Upstream/CD-
- R20 pad 1: /LEDs/RGB_IN -> /uController/RGB_DOUT
- SW30 pad 2: /Switches/COL5] -> /Column Decoder/COL[5]
- SW31 pad 2: /Switches/COL5] -> /Column Decoder/COL[5]
- SW32 pad 2: /Switches/COL5] -> /Column Decoder/COL[5]
- SW33 pad 2: /Switches/COL5] -> /Column Decoder/COL[5]
- SW34 pad 2: /Switches/COL5] -> /Column Decoder/COL[5]
- U3 pad 1: /USB Downstream 0/USBD- -> /USB Downstream 1/USBD-
- U3 pad 3: /USB Downstream 1/USBD+ -> /USB Downstream 0/USBD+
- U3 pad 4: /USB Downstream 1/USBD- -> /USB Downstream 0/USBD-
- U3 pad 6: /USB Downstream 0/USBD+ -> /USB Downstream 1/USBD+
- U6 pad 12: /Column Decoder/COLA[1] -> /Column Decoder/COLA[4]
- U6 pad 18: /Column Decoder/COLA[2] -> /Column Decoder/COLA[3]
- U6 pad 19: /Switches/ROW[0] -> Net-(U6-Pad19)
- U6 pad 20: /Switches/ROW[1] -> Net-(U6-Pad20)
- U6 pad 21: /Switches/ROW[2] -> /Switches/ROW[0]
- U6 pad 22: /Switches/ROW[3] -> /Switches/ROW[1]
- U6 pad 25: /Switches/ROW[4] -> /Switches/ROW[2]
- U6 pad 26: Net-(U6-Pad26) -> /Switches/ROW[3]
- U6 pad 27: /Switches/ROW[5] -> /Switches/ROW[4]
- U6 pad 28: /Column Decoder/COLA[3] -> /Switches/ROW[5]
- U6 pad 29: /Column Decoder/COLA[4] -> /Column Decoder/COLA[2]
- U6 pad 30: /Column Decoder/COLA[5] -> /Column Decoder/COLA[1]
- U6 pad 31: /Misc/ENC_A[0] -> /Column Decoder/COLA[0]
- U6 pad 32: /Misc/ENC_B[0] -> /uController/RGB_DOUT
- U6 pad 40: /uController/RGB_DOUT -> Net-(U6-Pad40)
- U6 pad 8: /Column Decoder/COLA[0] -> /Column Decoder/COLA[5]
Routing:
- net +3V3: track 0.00 -> 164.6 mm, vias 0 -> 3
- net /Column Decoder/COL[5]: track 0.00 -> 158.3 mm, vias 0 -> 6
- net /Switches/ROW[5]: track 331.9 -> 483.5 mm, vias 24 -> 25
- net /uController/RGB_DOUT: track 0.00 -> 132.2 mm, vias 0 -> 1
- net /Switches/ROW[4]: track 299.6 -> 419.5 mm, vias 0 -> 2
- net Net-(D14-Pad2): track 0.00 -> 105.1 mm, vias 0 -> 2
- net /Column Decoder/COL[8]: track 121.7 -> 226.5 mm, vias 6 -> 7
- net /Column Decoder/COLA[3]: track 0.00 -> 104.3 mm
- net /Column Decoder/COLA[5]: track 0.00 -> 102.2 mm
- net /Switches/COL5]: track 101.2 -> 0.00 mm, vias 5 -> 0
- net /Column Decoder/COLA[4]: track 0.00 -> 101.1 mm
- net /Column Decoder/COL[7]: track 101.2 -> 197.8 mm, vias 5 -> 6
- net /Column Decoder/COL[0]: track 106.8 -> 203.0 mm, vias 6 -> 7
- net /Switches/ROW[3]: track 327.5 -> 421.4 mm, vias 27 -> 29
- net /Column Decoder/COLA[0]: track 0.00 -> 90.6 mm
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- added copper zone on F.Cu, net +3V3
Other:
- board size 358.8 x 141.1 mm -> 358.8 x 150.8 mm

Commit message: Power supply routed
Parts:
- removed R7: 330R, resistor_smd:R_0603_1608Metric
- added C119: 100nF, Capacitor_smd:C_0603_1608Metric, F.Cu at (260.1, 62.7)
- added C120: 1uF, Capacitor_smd:C_0603_1608Metric, F.Cu at (231.7, 76.5)
- added C121: 47uF, Capacitor_smd:C_1210_3225Metric, F.Cu at (243.2, 61.9)
- added D194: LED, Diode_SMD:D_0603_1608Metric, F.Cu at (234.8, 47.5)
- added H10: MountingHole_Pad, mounting_hole:MountingHole_3.2mm_M3_ISO7380_Pad, F.Cu at (258.9, -20.4)
- added H11: MountingHole_Pad, mounting_hole:MountingHole_3.2mm_M3_ISO7380_Pad, F.Cu at (266.2, -27.7)
- added H12: MountingHole_Pad, mounting_hole:MountingHole_3.2mm_M3_ISO7380_Pad, F.Cu at (266.2, -20.4)
- added H5: MountingHole_Pad, mounting_hole:MountingHole_3.2mm_M3_ISO7380_Pad, F.Cu at (244.4, -27.7)
- added H6: MountingHole_Pad, mounting_hole:MountingHole_3.2mm_M3_ISO7380_Pad, F.Cu at (244.4, -20.4)
- added H7: MountingHole_Pad, mounting_hole:MountingHole_3.2mm_M3_ISO7380_Pad, F.Cu at (251.7, -27.7)
- added H8: MountingHole_Pad, mounting_hole:MountingHole_3.2mm_M3_ISO7380_Pad, F.Cu at (251.7, -20.4)
- added H9: MountingHole_Pad, mounting_hole:MountingHole_3.2mm_M3_ISO7380_Pad, F.Cu at (258.9, -27.7)
- added J7: Barrel_Jack_MountingPin, Connector_BarrelJack:BarrelJack_Wuerth_6941xx301002, F.Cu at (276.8, 65.8)
- added J8: Conn_01x03_Male, Connector_PinHeader_2.54mm:PinHeader_1x03_P2.54mm_Vertical, F.Cu at (237.3, 67.0)
- added L2: L, Inductor_SMD:L_10.4x10.4_H4.8, F.Cu at (251.3, 65.9)
- added R3: 330R, resistor_smd:R_0603_1608Metric, F.Cu at (234.3, 45.6)
- added U9: TCR2EF33, custom_footprint_library:TCR2EF33_SOT25, F.Cu at (230.8, 72.4)
- C4: value 100nF -> 10uF
- C45, R38, R39: moved to F.Cu
- C5: value 1uF -> 100nF
- D1: value LED -> D; footprint Diode_SMD:D_0603_1608Metric -> custom_footprint_library:DO-214AC
- R22, R23, R24, R25, R26, R27, R28, R29, R32, R33, R34, R35, R36, R37, R8, R9: value 4K7 -> 10K
- U2: value TCR2EF33 -> ADP2303ARDZ-5.0; footprint custom_footprint_library:TCR2EF33_SOT25 -> Package_SO:SOIC-8-1EP_3.9x4.9mm_P1.27mm_EP2.29x3mm
- moved D1 200.7 mm to (259.2, 65.6)
- moved R30 156.2 mm to (191.3, 63.1)
- moved R31 152.1 mm to (189.6, 63.1)
- moved C4 42.0 mm to (267.3, 58.9), turned to 90 degrees
- moved J5 41.4 mm to (196.6, 75.7), turned to 180 degrees
- moved SW1 35.0 mm to (200.2, 72.5), turned to 270 degrees
- moved U2 33.1 mm to (261.8, 59.0)
- moved R22 26.9 mm to (195.9, 68.4), turned to 0 degrees
- moved U1 20.0 mm to (215.6, 58.6), turned to 270 degrees
- moved R11 17.6 mm to (195.2, 41.6)
- moved R8 17.6 mm to (195.2, 38.4)
- moved R9 17.6 mm to (195.2, 40.0)
- moved R1 17.1 mm to (227.0, 44.0)
- moved C8 17.0 mm to (191.9, 39.7)
- moved C7 17.0 mm to (190.1, 39.6)
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Connections:
- C3 pad 1: +5V -> +5V0_USB
- C4 pad 1: +5V -> /Power/DCDC_IN
- C5 pad 1: +3V3 -> +5V
- D1 pad 1: Net-(D1-Pad1) -> /Power/SW
- D1 pad 2: +3V3 -> GND
- FB3 pad 1: +5V -> +5V0_USB
- U2 pad 1: +5V -> Net-(C119-Pad1)
- U2 pad 2: GND -> /Power/DCDC_IN
- U2 pad 3: +5V -> /Power/DCDC_IN
- U2 pad 5: +3V3 -> +5V0_EXT
- U6 pad 1: /Misc/SCL -> /Column Decoder/COLA[5]
- U6 pad 18: /Column Decoder/COLA[3] -> Net-(U6-Pad18)
- U6 pad 19: Net-(U6-Pad19) -> /Switches/ROW[0]
- U6 pad 20: Net-(U6-Pad20) -> /Switches/ROW[1]
- U6 pad 21: /Switches/ROW[0] -> /Switches/ROW[3]
- U6 pad 22: /Switches/ROW[1] -> /Switches/ROW[2]
- U6 pad 25: /Switches/ROW[2] -> /Switches/ROW[4]
- U6 pad 26: /Switches/ROW[3] -> /Switches/ROW[5]
- U6 pad 27: /Switches/ROW[4] -> /Column Decoder/COLA[2]
- U6 pad 28: /Switches/ROW[5] -> /Column Decoder/COLA[1]
- U6 pad 29: /Column Decoder/COLA[2] -> /Column Decoder/COLA[0]
- U6 pad 30: /Column Decoder/COLA[1] -> /uController/RGB_DOUT
- U6 pad 31: /Column Decoder/COLA[0] -> /Misc/SDA
- U6 pad 32: /uController/RGB_DOUT -> /Misc/SCL
- U6 pad 40: Net-(U6-Pad40) -> /Misc/ENC_B[0]
- U6 pad 41: /Misc/SDA -> /Misc/ENC_A[0]
- U6 pad 8: /Column Decoder/COLA[5] -> /Column Decoder/COLA[3]
Routing:
- net /Misc/SDA: track 0.00 -> 155.7 mm, vias 0 -> 1
- net /Misc/SCL: track 0.00 -> 153.1 mm, vias 0 -> 1
- net /Column Decoder/COLA[5]: track 102.2 -> 0.97 mm
- net /Switches/ROW[4]: track 419.5 -> 438.2 mm
- net /Switches/ROW[3]: track 421.4 -> 437.0 mm, vias 29 -> 28
- net RST: track 0.00 -> 13.8 mm, vias 0 -> 1
- net GND: track 60.3 -> 73.4 mm, vias 33 -> 43
- net /Switches/ROW[2]: track 397.9 -> 409.3 mm
- net /USB HUB/USB_DOWNSTREAM_LOCAL_OUT+: track 10.6 -> 20.5 mm, vias 1 -> 2
- net /USB HUB/USB_DOWNSTREAM_LOCAL_OUT-: track 10.3 -> 20.0 mm, vias 1 -> 2
- net /Switches/ROW[5]: track 483.5 -> 492.4 mm
- net Net-(C1-Pad2): track 18.5 -> 27.4 mm
- net VBUS: track 10.5 -> 19.3 mm
- net /Switches/ROW[0]: track 346.3 -> 355.1 mm
- net /Switches/ROW[1]: track 363.7 -> 371.7 mm
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- added copper zone on F.Cu, net +5V0_EXT
- added copper zone on F.Cu, net +5V0_USB
- added copper zone on F.Cu, net /Power/DCDC_IN
- added copper zone on F.Cu, net /Power/SW
